File: schematics/kicad/pico-glitcher.kicad_pcb (KiCad board)
At the start: 2 copper layers, 89.8 x 58.4 mm, 72 parts, among them Q1 IRLML2502, Q2 IRF7807PBF, Q3 TPS 79318, Q4 TPS2041, U1 NH245, U2 NH245, X1 BU-SMA, X2 BU-SMA, X3 M08X2

Commit message: Playing around.
Other:
- board text removed: "Pico Glitcher v1.1 (c) 2024 Matthias Kesenheimer"
Changed lines of the file:
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@@
 		(tags "SOIC SO")
 		(property "Reference" "Q2"
-			(at 0.076 3.556 360)
+			(at 0.076 3.556 0)
 			(layer "F.SilkS")
 			(effects
@@
 		)
 		(property "Value" "IRF7807PBF"
-			(at 0 3.4 360)
+			(at 0 3.4 0)
 			(layer "F.Fab")
 			(effects
@@
 		)
 		(fp_text user "${REFERENCE}"
-			(at 0 0 360)
+			(at 0 0 0)
 			(layer "F.Fab")
 			(effects
@@
 		(descr "Ultraminiature Surface Mount Slide Switch, right-angle, https://www.ckswitches.com/media/1424/pcm.pdf")
 		(property "Reference" "S1"
-			(at 6.68 0.508 360)
+			(at 6.68 0.508 0)
 			(layer "F.SilkS")
 			(effects
@@
 		)
 		(property "Value" "Micro Slide Switch"
-			(at 0 4.25 360)
+			(at 0 4.25 0)
 			(layer "F.Fab")
 			(effects
@@
 		)
 		(fp_text user "${REFERENCE}"
-			(at 0 -3.2 360)
+			(at 0 -3.2 0)
 			(layer "F.Fab")
 			(effects
@@
 		)
 		(pad "1" smd rect
-			(at -1.8 0.2 270)
+			(at 1.9 0.2 270)
 			(size 2.2 0.65)
 			(layers "F.Cu" "F.Paste" "F.Mask")
@@
 		)
 		(pad "2" smd rect
-			(at 1.9 0.2 270)
+			(at -1.8 0.2 270)
 			(size 2.2 0.65)
 			(layers "F.Cu" "F.Paste" "F.Mask")
@@
 		)
 	)
-	(gr_text "Pico Glitcher v1.1\n(c) 2024 Matthias Kesenheimer"
-		(at 147.1931 110.8406 0)
-		(layer "F.SilkS")
-		(effects
-			(font
-				(size 1.2 1.2)
-				(thickness 0.15)
-			)
-			(justify left bottom)
-		)
-	)
